File: turbo_86m_extender_board.kicad_sch (KiCad schematic)
At the start: 0 parts

Commit message: Initial upload
Parts:
- added D1, D2, D3, D4: SNP96, Turbo:snp59_96_female_angle, symbol Turbo86m:SNP96
Connections:
- new net A1: D1.1 (A1), D2.32 (A32)
- new net A10: D1.10 (A10), D2.23 (A23)
- new net A11: D1.11 (A11), D2.22 (A22)
- new net A12: D1.12 (A12), D2.21 (A21)
- new net A13: D1.13 (A13), D2.20 (A20)
- new net A14: D1.14 (A14), D2.19 (A19)
- new net A15: D1.15 (A15), D2.18 (A18)
- new net A16: D1.16 (A16), D2.17 (A17)
- new net A17: D1.17 (A17), D2.16 (A16)
- new net A18: D1.18 (A18), D2.15 (A15)
- new net A19: D1.19 (A19), D2.14 (A14)
- new net A2: D1.2 (A2), D2.31 (A31)
- new net A20: D1.20 (A20), D2.13 (A13)
- new net A21: D1.21 (A21), D2.12 (A12)
- new net A22: D1.22 (A22), D2.11 (A11)
- new net A23: D1.23 (A23), D2.10 (A10)
- new net A24: D1.24 (A24), D2.9 (A9)
- new net A25: D1.25 (A25), D2.8 (A8)
- new net A26: D1.26 (A26), D2.7 (A7)
- new net A27: D1.27 (A27), D2.6 (A6)
- new net A28: D1.28 (A28), D2.5 (A5)
- new net A29: D1.29 (A29), D2.4 (A4)
- new net A3: D1.3 (A3), D2.30 (A30)
- new net A30: D1.30 (A30), D2.3 (A3)
- new net A31: D1.31 (A31), D2.2 (A2)
- new net A32: D1.32 (A32), D2.1 (A1)
- new net A4: D1.4 (A4), D2.29 (A29)
- new net A5: D1.5 (A5), D2.28 (A28)
- new net A6: D1.6 (A6), D2.27 (A27)
- new net A7: D1.7 (A7), D2.26 (A26)
- new net A8: D1.8 (A8), D2.25 (A25)
- new net A9: D1.9 (A9), D2.24 (A24)
- new net B1: D1.33 (B1), D2.64 (B32)
- new net B10: D1.42 (B10), D2.55 (B23)
- new net B11: D1.43 (B11), D2.54 (B22)
- new net B12: D1.44 (B12), D2.53 (B21)
- new net B13: D1.45 (B13), D2.52 (B20)
- new net B14: D1.46 (B14), D2.51 (B19)
- new net B15: D1.47 (B15), D2.50 (B18)
- new net B16: D1.48 (B16), D2.49 (B17)
- new net B17: D1.49 (B17), D2.48 (B16)
- new net B18: D1.50 (B18), D2.47 (B15)
- new net B19: D1.51 (B19), D2.46 (B14)
- new net B2: D1.34 (B2), D2.63 (B31)
- new net B20: D1.52 (B20), D2.45 (B13)
- new net B21: D1.53 (B21), D2.44 (B12)
- new net B22: D1.54 (B22), D2.43 (B11)
- new net B23: D1.55 (B23), D2.42 (B10)
- new net B24: D1.56 (B24), D2.41 (B9)
- new net B25: D1.57 (B25), D2.40 (B8)
- new net B26: D1.58 (B26), D2.39 (B7)
- new net B27: D1.59 (B27), D2.38 (B6)
- new net B28: D1.60 (B28), D2.37 (B5)
- new net B29: D1.61 (B29), D2.36 (B4)
- new net B3: D1.35 (B3), D2.62 (B30)
- new net B30: D1.62 (B30), D2.35 (B3)
- new net B31: D1.63 (B31), D2.34 (B2)
- new net B32: D1.64 (B32), D2.33 (B1)
- new net B4: D1.36 (B4), D2.61 (B29)
- new net B5: D1.37 (B5), D2.60 (B28)
- new net B6: D1.38 (B6), D2.59 (B27)
- new net B7: D1.39 (B7), D2.58 (B26)
- new net B8: D1.40 (B8), D2.57 (B25)
- new net B9: D1.41 (B9), D2.56 (B24)
- new net C1: D1.65 (C1), D2.96 (C32)
- new net C10: D1.74 (C10), D2.87 (C23)
- new net C11: D1.75 (C11), D2.86 (C22)
- new net C12: D1.76 (C12), D2.85 (C21)
- new net C13: D1.77 (C13), D2.84 (C20)
- new net C14: D1.78 (C14), D2.83 (C19)
- new net C15: D1.79 (C15), D2.82 (C18)
- new net C16: D1.80 (C16), D2.81 (C17)
- new net C17: D1.81 (C17), D2.80 (C16)
- new net C18: D1.82 (C18), D2.79 (C15)
- new net C19: D1.83 (C19), D2.78 (C14)
- new net C2: D1.66 (C2), D2.95 (C31)
- new net C20: D1.84 (C20), D2.77 (C13)
- new net C21: D1.85 (C21), D2.76 (C12)
- new net C22: D1.86 (C22), D2.75 (C11)
- new net C23: D1.87 (C23), D2.74 (C10)
- new net C24: D1.88 (C24), D2.73 (C9)
- new net C25: D1.89 (C25), D2.72 (C8)
- new net C26: D1.90 (C26), D2.71 (C7)
- new net C27: D1.91 (C27), D2.70 (C6)
- new net C28: D1.92 (C28), D2.69 (C5)
- new net C29: D1.93 (C29), D2.68 (C4)
- new net C3: D1.67 (C3), D2.94 (C30)
- new net C30: D1.94 (C30), D2.67 (C3)
- new net C31: D1.95 (C31), D2.66 (C2)
- new net C32: D1.96 (C32), D2.65 (C1)
- new net C4: D1.68 (C4), D2.93 (C29)
- new net C5: D1.69 (C5), D2.92 (C28)
- new net C6: D1.70 (C6), D2.91 (C27)
- new net C7: D1.71 (C7), D2.90 (C26)
- new net C8: D1.72 (C8), D2.89 (C25)
- new net C9: D1.73 (C9), D2.88 (C24)
- new net _A1: D3.1 (A1), D4.32 (A32)
- new net _A10: D3.10 (A10), D4.23 (A23)
- new net _A11: D3.11 (A11), D4.22 (A22)
- new net _A12: D3.12 (A12), D4.21 (A21)
- new net _A13: D3.13 (A13), D4.20 (A20)
- new net _A14: D3.14 (A14), D4.19 (A19)
- new net _A15: D3.15 (A15), D4.18 (A18)
- new net _A16: D3.16 (A16), D4.17 (A17)
- new net _A17: D3.17 (A17), D4.16 (A16)
- new net _A18: D3.18 (A18), D4.15 (A15)
- new net _A19: D3.19 (A19), D4.14 (A14)
- new net _A2: D3.2 (A2), D4.31 (A31)
- new net _A20: D3.20 (A20), D4.13 (A13)
- new net _A21: D3.21 (A21), D4.12 (A12)
- new net _A22: D3.22 (A22), D4.11 (A11)
- new net _A23: D3.23 (A23), D4.10 (A10)
- new net _A24: D3.24 (A24), D4.9 (A9)
- new net _A25: D3.25 (A25), D4.8 (A8)
- new net _A26: D3.26 (A26), D4.7 (A7)
- new net _A27: D3.27 (A27), D4.6 (A6)
- new net _A28: D3.28 (A28), D4.5 (A5)
- new net _A29: D3.29 (A29), D4.4 (A4)
- new net _A3: D3.3 (A3), D4.30 (A30)
- new net _A30: D3.30 (A30), D4.3 (A3)
- new net _A31: D3.31 (A31), D4.2 (A2)
- new net _A32: D3.32 (A32), D4.1 (A1)
- new net _A4: D3.4 (A4), D4.29 (A29)
- new net _A5: D3.5 (A5), D4.28 (A28)
- new net _A6: D3.6 (A6), D4.27 (A27)
- new net _A7: D3.7 (A7), D4.26 (A26)
- new net _A8: D3.8 (A8), D4.25 (A25)
- new net _A9: D3.9 (A9), D4.24 (A24)
- new net _B1: D3.33 (B1), D4.64 (B32)
- new net _B10: D3.42 (B10), D4.55 (B23)
- new net _B11: D3.43 (B11), D4.54 (B22)
- new net _B12: D3.44 (B12), D4.53 (B21)
- new net _B13: D3.45 (B13), D4.52 (B20)
- new net _B14: D3.46 (B14), D4.51 (B19)
- new net _B15: D3.47 (B15), D4.50 (B18)
- new net _B16: D3.48 (B16), D4.49 (B17)
- new net _B17: D3.49 (B17), D4.48 (B16)
- new net _B18: D3.50 (B18), D4.47 (B15)
- new net _B19: D3.51 (B19), D4.46 (B14)
- new net _B2: D3.34 (B2), D4.63 (B31)
- new net _B20: D3.52 (B20), D4.45 (B13)
- new net _B21: D3.53 (B21), D4.44 (B12)
- new net _B22: D3.54 (B22), D4.43 (B11)
- new net _B23: D3.55 (B23), D4.42 (B10)
- new net _B24: D3.56 (B24), D4.41 (B9)
- new net _B25: D3.57 (B25), D4.40 (B8)
- new net _B26: D3.58 (B26), D4.39 (B7)
- new net _B27: D3.59 (B27), D4.38 (B6)
- new net _B28: D3.60 (B28), D4.37 (B5)
- new net _B29: D3.61 (B29), D4.36 (B4)
- new net _B3: D3.35 (B3), D4.62 (B30)
- new net _B30: D3.62 (B30), D4.35 (B3)
- new net _B31: D3.63 (B31), D4.34 (B2)
- new net _B32: D3.64 (B32), D4.33 (B1)
- new net _B4: D3.36 (B4), D4.61 (B29)
- new net _B5: D3.37 (B5), D4.60 (B28)
- new net _B6: D3.38 (B6), D4.59 (B27)
- new net _B7: D3.39 (B7), D4.58 (B26)
- new net _B8: D3.40 (B8), D4.57 (B25)
- new net _B9: D3.41 (B9), D4.56 (B24)
- new net _C1: D3.65 (C1), D4.96 (C32)
- new net _C10: D3.74 (C10), D4.87 (C23)
- new net _C11: D3.75 (C11), D4.86 (C22)
- new net _C12: D3.76 (C12), D4.85 (C21)
- new net _C13: D3.77 (C13), D4.84 (C20)
- new net _C14: D3.78 (C14), D4.83 (C19)
- new net _C15: D3.79 (C15), D4.82 (C18)
- new net _C16: D3.80 (C16), D4.81 (C17)
- new net _C17: D3.81 (C17), D4.80 (C16)
- new net _C18: D3.82 (C18), D4.79 (C15)
- new net _C19: D3.83 (C19), D4.78 (C14)
- new net _C2: D3.66 (C2), D4.95 (C31)
- new net _C20: D3.84 (C20), D4.77 (C13)
- new net _C21: D3.85 (C21), D4.76 (C12)
- new net _C22: D3.86 (C22), D4.75 (C11)
- new net _C23: D3.87 (C23), D4.74 (C10)
- new net _C24: D3.88 (C24), D4.73 (C9)
- new net _C25: D3.89 (C25), D4.72 (C8)
- new net _C26: D3.90 (C26), D4.71 (C7)
- new net _C27: D3.91 (C27), D4.70 (C6)
- new net _C28: D3.92 (C28), D4.69 (C5)
- new net _C29: D3.93 (C29), D4.68 (C4)
- new net _C3: D3.67 (C3), D4.94 (C30)
- new net _C30: D3.94 (C30), D4.67 (C3)
- new net _C31: D3.95 (C31), D4.66 (C2)
- new net _C32: D3.96 (C32), D4.65 (C1)
- new net _C4: D3.68 (C4), D4.93 (C29)
- new net _C5: D3.69 (C5), D4.92 (C28)
- new net _C6: D3.70 (C6), D4.91 (C27)
- new net _C7: D3.71 (C7), D4.90 (C26)
- new net _C8: D3.72 (C8), D4.89 (C25)
- new net _C9: D3.73 (C9), D4.88 (C24)
