File: turbo_86m_extender_board.kicad_pcb (KiCad board)
At the start: 2 copper layers, 1 part

Commit message: Initial upload
Parts:
- removed REF**: snp59_96_female_angle, Turbo:snp59_96_female_angle
- added D1: SNP96, Turbo:snp59_96_female_angle, F.Cu at (11.0, 5.00)
- added D2: SNP96, Turbo:snp59_96_female_angle, F.Cu at (88.5, 214.0)
- added D3: SNP96, Turbo:snp59_96_female_angle, F.Cu at (143.5, 5.00)
- added D4: SNP96, Turbo:snp59_96_female_angle, F.Cu at (221.0, 214.0)
Routing:
- net A30: track 0.00 -> 210.2 mm
- net A7: track 0.00 -> 210.1 mm
- net A32: track 0.00 -> 210.1 mm
- net A28: track 0.00 -> 210.1 mm
- net A22: track 0.00 -> 210.1 mm
- net A10: track 0.00 -> 210.1 mm
- net _A5: track 0.00 -> 210.1 mm
- net _A20: track 0.00 -> 210.1 mm
- net A8: track 0.00 -> 210.1 mm
- net A4: track 0.00 -> 210.1 mm
- net A26: track 0.00 -> 210.1 mm
- net A24: track 0.00 -> 210.1 mm
- net A12: track 0.00 -> 210.1 mm
- net A11: track 0.00 -> 210.1 mm
- net _A9: track 0.00 -> 209.9 mm
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Other:
- board outline added: 232 x 219 mm

Commit message: Ver. 0.1
Parts:
- added G***: LOGO, Turbo:logo_3, F.Cu at (116.6, 54.2)
- added G***: LOGO, Turbo:logo_1, F.Cu at (116.8, 115.5)
- added G***: LOGO, Turbo:logo_2, F.Cu at (116.6, 175.0)

Commit message: Update turbo_86m_extender_board.kicad_pcb
Parts:
- moved D2 30.0 mm to (88.5, 244.0)
- moved D4 30.0 mm to (221.0, 244.0)
Routing:
- net _B15: track 204.9 -> 235.2 mm
- net _A1: track 209.9 -> 240.1 mm
- net _A26: track 209.9 -> 240.1 mm
- net _A23: track 209.9 -> 240.1 mm
- net _A22: track 209.9 -> 240.1 mm
- net _A11: track 209.9 -> 240.1 mm
- net _A9: track 209.9 -> 240.1 mm
- net _A7: track 209.9 -> 240.1 mm
- net _A29: track 209.9 -> 240.1 mm
- net _A25: track 209.9 -> 240.1 mm
- net _A21: track 209.9 -> 240.1 mm
- net _B30: track 204.9 -> 234.9 mm
- net _B26: track 204.9 -> 234.9 mm
- net _A5: track 210.1 -> 240.1 mm
- net _A28: track 209.9 -> 239.9 mm
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Other:
- board size 232 x 219 mm -> 232 x 249 mm
